File: 01_main-board/Dumpling_Main.kicad_pcb (KiCad board)
At the start: 4 copper layers, 353 parts, among them J1 Conn_ARM_SWD_TagConnect_TC203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, J10 MICROMOD-2222-C, J11 USB_C_Receptacle_USB2.0_16P, J12 Conn_ARM_SWD_TagConnect_TC203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, J13 MICROMOD-2222-C, J14 USB_C_Receptacle_USB2.0_16P, J15 Conn_ARM_SWD_TagConnect_TC203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, J16 MICROMOD-2222-C, J17 USB_C_Receptacle_USB2.0_16P, J18 Conn_ARM_SWD_TagConnect_TC203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, J19 MICROMOD-2222-C, J2 Micro_SD_Card, J20 USB_C_Receptacle_USB2.0_16P, J21 Conn_ARM_SWD_TagConnect_TC203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, J22 MICROMOD-2222-C, J23 USB_C_Receptacle_USB2.0_16P, J3 USB_C_Receptacle_USB2.0_16P, J4 XT30PW-M, J6 Conn_ARM_SWD_TagConnect_TC203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, J7 MICROMOD-2222-C, J8 USB_C_Receptacle_USB2.0_16P, J9 Conn_ARM_SWD_TagConnect_TC203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, Q1 AO3401A, Q2 S8050, SW1 SW_DPST, SW10 SW_SPDT, SW11 SW_DPST, SW12 SW_SPDT, SW13 SW_DPST, SW14 SW_SPDT, SW2 SW_DPST, SW3 SW_DPST, SW4 SW_SPDT, SW5 SW_DPST, SW6 SW_SPDT, SW7 SW_DPST, SW8 SW_SPDT, SW9 SW_DPST, U1 STM32F405RGTx, U10 W25Q128JVS, U11 USBLC6-2SC6, U12 W25Q128JVS, U13 STM32F411CEUx, U14 USBLC6-2SC6, U15 W25Q128JVS, U16 STM32F411CEUx, U17 USBLC6-2SC6, U18 W25Q128JVS, U19 STM32F411CEUx, U2 USBLC6-2SC6, U20 USBLC6-2SC6, U22 STM32F411CEUx, U23 USBLC6-2SC6, U24 W25Q128JVS, U25 TPS562200, U26 TPS562200, U3 W25Q128JVS, U4 STM32F411CEUx, U5 STM32F411CEUx, U6 USBLC6-2SC6, U7 INA219AxD, U8 W25Q128JVS, Y1 32.768kHz, Y2 32.768kHz, Y3 32.768kHz, Y4 32.768kHz, Y5 32.768kHz, Y6 32.768kHz, Y7 32.768kHz

Commit message: layout
Parts:
- moved D4 30.7 mm to (108.2, 90.0), turned to 90 degrees
- moved TP32 29.6 mm to (81.7, 73.0), turned to 0 degrees
- moved TP31 27.9 mm to (80.0, 74.5), turned to 0 degrees
- moved SW4 26.0 mm to (104.5, 90.0), turned to 0 degrees
- moved TP28 25.4 mm to (81.7, 76.0), turned to 0 degrees
- moved C14 23.8 mm to (100.2, 90.1)
- moved SW3 23.8 mm to (97.3, 90.1)
- moved TP30 23.8 mm to (80.0, 77.5), turned to 0 degrees
- moved R11 23.2 mm to (105.3, 86.5), turned to 0 degrees
- moved R10 22.1 mm to (105.0, 85.3), turned to 180 degrees
- moved TP19 21.2 mm to (81.7, 79.0), turned to 0 degrees
- moved TP12 19.7 mm to (80.0, 80.5), turned to 0 degrees
- moved TP24 17.1 mm to (81.7, 82.0), turned to 0 degrees
- moved R14 12.1 mm to (111.0, 60.7), turned to -90 degrees
- moved C29 10.4 mm to (100.2, 63.9), turned to 0 degrees
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Routing:
- net Net-(J8-CC2): track 0.00 -> 9.59 mm
- net co1_OSC_IN: track 2.46 -> 10.8 mm
- net Net-(J8-CC1): track 0.00 -> 7.15 mm
- net GND: track 5.88 -> 10.8 mm
- net co1_OSC_OUT: track 0.00 -> 4.04 mm
- net Net-(SW4-B): track 5.59 -> 3.59 mm
- net co1_FLASH_WP: track 0.00 -> 1.76 mm
- net +3V3: track 5.82 -> 7.44 mm
- net co1_NRST: track 0.00 -> 1.39 mm
- net co1_USB_D+_ESD: track 10.1 -> 11.2 mm
- net Net-(D4-A): track 3.14 -> 4.23 mm
