File: 01_main-board/Dumpling_Main.kicad_pcb (KiCad board)
At the start: 4 copper layers, 75 x 135.2 mm, 354 parts, among them J1 Conn_ARM_SWD_TagConnect_TC203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, J10 MICROMOD-2222-C, J11 USB_C_Receptacle_USB2.0_16P, J12 Conn_ARM_SWD_TagConnect_TC203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, J13 MICROMOD-2222-C, J14 USB_C_Receptacle_USB2.0_16P, J15 Conn_ARM_SWD_TagConnect_TC203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, J16 MICROMOD-2222-C, J17 USB_C_Receptacle_USB2.0_16P, J18 Conn_ARM_SWD_TagConnect_TC203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, J19 MICROMOD-2222-C, J2 Micro_SD_Card, J20 USB_C_Receptacle_USB2.0_16P, J21 Conn_ARM_SWD_TagConnect_TC203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, J22 MICROMOD-2222-C, J23 USB_C_Receptacle_USB2.0_16P, J3 USB_C_Receptacle_USB2.0_16P, J4 XT30PW-M, J5 SM04B-SRSS-TB, J6 Conn_ARM_SWD_TagConnect_TC203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, J7 MICROMOD-2222-C, J8 USB_C_Receptacle_USB2.0_16P, J9 Conn_ARM_SWD_TagConnect_TC203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, Q1 AO3401A, Q2 S8050, SW1 SW_DPST, SW10 SW_SPDT, SW11 SW_DPST, SW12 SW_SPDT, SW13 SW_DPST, SW14 SW_SPDT, SW2 SW_DPST, SW3 SW_DPST, SW4 SW_SPDT, SW5 SW_DPST, SW6 SW_SPDT, SW7 SW_DPST, SW8 SW_SPDT, SW9 SW_DPST, U1 STM32F405RGTx, U10 W25Q128JVS, U11 USBLC6-2SC6, U12 W25Q128JVS, U13 STM32F411CEUx, U14 USBLC6-2SC6, U15 W25Q128JVS, U16 STM32F411CEUx, U17 USBLC6-2SC6, U18 W25Q128JVS, U19 STM32F411CEUx, U2 USBLC6-2SC6, U20 USBLC6-2SC6, U22 STM32F411CEUx, U23 USBLC6-2SC6, U24 W25Q128JVS, U25 TPS562200, U26 TPS562200, U3 W25Q128JVS, U4 STM32F411CEUx, U5 STM32F411CEUx, U6 USBLC6-2SC6, U8 W25Q128JVS, U9 INA219AxDCN, Y1 32.768kHz, Y2 32.768kHz, Y3 32.768kHz, Y4 32.768kHz, Y5 32.768kHz, Y6 32.768kHz, Y7 32.768kHz

Commit message: Update Dumpling_Main.kicad_pcb
Parts:
- moved VBAT1 1.90 mm to (80.5, 52.0)
Changed lines of the file:
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@@
 	(footprint "TestPoint:TestPoint_Pad_D1.5mm"
 		(layer "F.Cu")
-		(at 82.4 52.05)
+		(at 80.5 52)
 		(descr "SMD pad as test Point, diameter 1.5mm")
 		(tags "test point SMD pad")

Commit message: wired
Parts:
- added C105: 10n, Capacitor_SMD:C_0402_1005Metric, F.Cu at (145.4, 53.9)
- added C106: 0.22u, Capacitor_SMD:C_0402_1005Metric, F.Cu at (147.3, 53.9)
- added C107: 0.22u, Capacitor_SMD:C_0402_1005Metric, F.Cu at (147.7, 47.4)
- added R80: 4.7k, Resistor_SMD:R_0402_1005Metric, F.Cu at (153.7, 63.1)
- added R81: 4.7k, Resistor_SMD:R_0402_1005Metric, F.Cu at (153.7, 62.2)
- added R82: 5.1k, Resistor_SMD:R_0402_1005Metric, F.Cu at (142.8, 52.2)
- added R83: 5.1k, Resistor_SMD:R_0402_1005Metric, F.Cu at (143.6, 53.9)
- added R84: 10k, Resistor_SMD:R_0402_1005Metric, F.Cu at (149.1, 52.2)
- added U7: MPU-6050, Sensor_Motion:InvenSense_QFN-24_4x4mm_P0.5mm, F.Cu at (145.9, 50.5)
- TP1, TP10, TP11, TP2, TP3, TP4, TP5, TP6, TP7, TP8, TP9, VBAT1, VBUS1, VIN1: moved to B.Cu
- moved VBAT1 25.3 mm to (98.8, 69.4)
- moved C100 23.8 mm to (147.9, 163.8)
- moved C84 22.9 mm to (113.6, 163.8), turned to 180 degrees
- moved C58 22.9 mm to (113.6, 128.6), turned to 180 degrees
- moved C62 21.5 mm to (128.9, 112.5), turned to -90 degrees
- moved C91 21.5 mm to (128.9, 147.7), turned to -90 degrees
- moved C97 21.3 mm to (164.6, 147.7), turned to -90 degrees
- moved VBUS1 19.6 mm to (98.8, 66.3)
- moved VIN1 16.9 mm to (98.8, 63.3)
- moved C78 13.7 mm to (147.9, 128.7), turned to -90 degrees
- moved C49 13.1 mm to (147.9, 92.6), turned to -90 degrees
- moved TP4 12.2 mm to (67.1, 50.5)
- moved TP8 12.2 mm to (70.7, 50.5)
- moved C46 12.0 mm to (156.9, 83.2), turned to 0 degrees
- moved C71 11.4 mm to (157.0, 119.2), turned to 0 degrees
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Connections:
- J2 pad 8: SDIO_D1 -> SDIO_D7
- U1 pad 38: unconnected-(U1-PC7-Pad38) -> SDIO_D7
- U1 pad 40: SDIO_D1 -> I2C3_SDA
- U1 pad 41: unconnected-(U1-PA8-Pad41) -> I2C3_SCL
- U1 pad 42: unconnected-(U1-PA9-Pad42) -> IMU_INT
Routing:
- net SPI2_MOSI: track 0.00 -> 243.7 mm, vias 0 -> 7
- net SPI2_SCK: track 0.00 -> 238.8 mm, vias 0 -> 7
- net SPI2_MISO: track 0.00 -> 238.5 mm, vias 0 -> 7
- net I2C2_SCL: track 3.06 -> 230.1 mm, vias 0 -> 7
- net Trigger: track 17.7 -> 241.9 mm, vias 6 -> 7
- net I2C2_SDA: track 2.90 -> 214.8 mm, vias 0 -> 7
- net co5_NRST: track 9.70 -> 168.9 mm, vias 0 -> 2
- net +5V: track 25.4 -> 173.2 mm, vias 7 -> 48
- net SPI2_NSS5: track 34.5 -> 178.2 mm
- net co6_NRST: track 9.70 -> 140.6 mm, vias 0 -> 2
- net SPI2_NSS6: track 34.3 -> 148.9 mm
- net co3_NRST: track 9.70 -> 117.4 mm, vias 0 -> 2
- net VBUS: track 57.7 -> 162.3 mm, vias 20 -> 21
- net co4_NRST: track 9.70 -> 98.8 mm, vias 0 -> 2
- net SPI2_NSS3: track 41.5 -> 122.4 mm
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- added copper zone on In2.Cu, net +3V3
- added copper zone on In2.Cu, net +5V
- added copper zone on In2.Cu, net VBUS
- added copper zone on In2.Cu, net VIN
Other:
- copper layers 4 -> 6
- board text added: "change switch, import 3d model, tp, Cu fill vias -> run drc -> label components"
- board text added: "no copper directly below component"
- board text removed: "RxTx"
- board text removed: "i2c1:INA"
- board text removed: "spi1:flsh"
- board text removed: "x:35.7 y: 35.2"

Commit message: wiring fin, pre-drc
Parts:
- moved TP4 100.3 mm to (164.5, 74.6)
- moved TP3 99.1 mm to (164.5, 72.6)
- moved TP8 95.7 mm to (164.5, 69.5), turned to 180 degrees
- moved TP7 94.8 mm to (164.5, 67.5), turned to 180 degrees
- moved TP6 94.2 mm to (164.5, 65.5), turned to 180 degrees
- moved TP5 93.9 mm to (164.5, 63.5), turned to 180 degrees
- moved TP11 90.5 mm to (164.5, 60.8), turned to 180 degrees
- moved TP9 90.4 mm to (164.5, 56.8), turned to 180 degrees
- moved TP10 90.3 mm to (164.5, 58.8), turned to 180 degrees
- moved TP2 36.5 mm to (98.8, 75.8), turned to 180 degrees
- moved TP1 34.0 mm to (98.8, 73.5), turned to 180 degrees
- moved VBAT1 0.10 mm to (98.8, 69.3)
Routing:
- net SPI1_NSS: track 25.0 -> 50.0 mm
- net SPI1_MISO: track 24.5 -> 48.8 mm
- net SPI1_SCK: track 16.9 -> 40.2 mm
- net SPI1_MOSI: track 18.3 -> 40.5 mm
- net SPI2_MOSI: track 243.7 -> 264.9 mm
- net I2C2_SCL: track 230.1 -> 250.1 mm
- net SPI2_MISO: track 238.5 -> 258.3 mm
- net SPI2_SCK: track 238.8 -> 257.1 mm
- net I2C2_SDA: track 214.8 -> 232.9 mm
- net GND: track 469.8 -> 465.1 mm, vias 164 -> 178
- net VIN: track 89.5 -> 86.4 mm, vias 22 -> 38
- net SDIO_CMD: track 27.8 -> 29.5 mm
- net co6_NRST: track 140.6 -> 138.9 mm
- net +3V3: track 246.0 -> 247.3 mm, vias 136 -> 134
- net +5V: track 173.2 -> 174.2 mm, vias 48 -> 42
- added copper zone on In1.Cu, net GND
Other:
- board text added: "change switch? -> run drc -> finish silkscreen"
- board text removed: "change switch, import 3d model, tp, Cu fill vias -> run drc -> label components"

Commit message: ebay backboard
Parts:
- removed MP1, MP2, MP3, MP4, MP5, MP6: ~, WA-SMSI_9774XXX151:WA-SMSI_9774025151
- added G***: LOGO, LOGO, F.Cu at (205.2, 71.0)
- added G***: LOGO, LOGO, F.Cu at (165.0, 140.0)
- added G***: LOGO, LOGO, F.Cu at (165.4, 104.3)
- added G***: LOGO, LOGO, F.Cu at (130.3, 139.9)
- added G***: LOGO, LOGO, F.Cu at (130.4, 104.0)
- added G***: LOGO, LOGO, B.Cu at (132.7, 59.3)
- added G***: LOGO, LOGO, B.Cu at (132.4, 73.2)
- added U21: SMTSOM2_525STR, SMTSOM2.525STR:SMD_BD5.6-D4.1, F.Cu at (162.9, 132.4)
- added U27: SMTSOM2_525STR, SMTSOM2.525STR:SMD_BD5.6-D4.1, F.Cu at (127.2, 132.4)
- added U28: SMTSOM2_525STR, SMTSOM2.525STR:SMD_BD5.6-D4.1, F.Cu at (127.0, 96.3)
- added U29: SMTSOM2_525STR, SMTSOM2.525STR:SMD_BD5.6-D4.1, F.Cu at (162.9, 167.6)
- added U30: SMTSOM2_525STR, SMTSOM2.525STR:SMD_BD5.6-D4.1, F.Cu at (127.2, 167.6)
- added U31: SMTSOM2_525STR, SMTSOM2.525STR:SMD_BD5.6-D4.1, F.Cu at (162.9, 96.4)
- BZ1: footprint CSS-0575B-SMT:CUI_CSS-0575B-SMT -> FST-5030:BUZ-SMD_FST-5030
- SW1: value SW_DPST -> SW_SPDT; footprint CJS-1200TA:SW_CJS-1200TA -> JS102011JCQN:SW_JS102011JCQN
- SW10, SW12, SW14, SW4, SW6, SW8: footprint CJS-1200TA:SW_CJS-1200TA -> JS102011JCQN:SW_JS102011JCQN
- SW11, SW13, SW2, SW3, SW5, SW7, SW9: value SW_DPST -> SW_SPST
- moved R2 3.86 mm to (139.7, 53.4)
- moved D17 3.81 mm to (160.2, 172.9), turned to 180 degrees
- moved D15 3.11 mm to (127.0, 176.5)
- moved D4 2.98 mm to (126.6, 106.0)
- moved D11 2.69 mm to (126.6, 141.9)
- moved D9 2.49 mm to (162.0, 106.0)
- moved D13 2.39 mm to (162.0, 141.7)
- moved SW1 2.18 mm to (134.5, 53.3)
- moved C34 1.74 mm to (111.8, 47.7)
- moved C38 1.74 mm to (113.8, 47.7)
- moved L2 1.74 mm to (108.5, 47.5)
- moved R16 1.74 mm to (108.1, 56.8)
- moved C31 1.74 mm to (103.2, 51.5)
- moved C32 1.74 mm to (105.2, 51.5)
- moved C33 1.74 mm to (110.8, 53.9)
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Connections:
- J11 pad B8: unconnected-(J11-SBU1-PadA8) -> unconnected-(J11-SBU2-PadB8)
- J14 pad B8: unconnected-(J14-SBU1-PadA8) -> unconnected-(J14-SBU2-PadB8)
- J17 pad B8: unconnected-(J17-SBU1-PadA8) -> unconnected-(J17-SBU2-PadB8)
- J20 pad B8: unconnected-(J20-SBU1-PadA8) -> unconnected-(J20-SBU2-PadB8)
- J23 pad B8: unconnected-(J23-SBU1-PadA8) -> unconnected-(J23-SBU2-PadB8)
- J8 pad B8: unconnected-(J8-SBU1-PadA8) -> unconnected-(J8-SBU2-PadB8)
Routing:
- net GND: track 465.1 -> 644.8 mm, vias 178 -> 257
- net NRST: track 29.6 -> 69.4 mm
- net co6_FLASH_HOLD: track 3.30 -> 41.2 mm, vias 1 -> 2
- net co4_FLASH_HOLD: track 3.30 -> 39.8 mm, vias 1 -> 2
- net co2_FLASH_HOLD: track 3.30 -> 38.6 mm, vias 1 -> 2
- net co2_FLASH_WP: track 3.62 -> 32.6 mm, vias 1 -> 2
- net co6_FLASH_WP: track 3.62 -> 31.5 mm, vias 1 -> 2
- net co4_FLASH_WP: track 3.62 -> 31.4 mm, vias 1 -> 2
- net co1_FLASH_HOLD: track 3.30 -> 28.3 mm, vias 1 -> 2
- net co5_FLASH_HOLD: track 3.30 -> 28.2 mm, vias 1 -> 2
- net co3_FLASH_HOLD: track 3.30 -> 28.1 mm, vias 1 -> 2
- net I2C1_SCL: track 38.8 -> 62.9 mm
- net Net-(SW1-B): track 4.95 -> 28.1 mm, vias 1 -> 2
- net I2C1_SDA: track 38.0 -> 60.9 mm
- net co1_FLASH_WP: track 3.62 -> 23.5 mm, vias 1 -> 2
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- added copper zone on B.Cu, net GND
- added copper zone on In3.Cu, net GND
- added copper zone on In4.Cu, net GND
Other:
- board text added: "1"
- board text added: "2"
- board text added: "3"
- board text added: "3V3"
- board text added: "4"
- board text added: "5"
- board text added: "5V"
- board text added: "6"
- board text added: "BOOT"
- board text added: "Data Dumpling Payload v0.1 04/25 @seoyoonij"
- board text added: "F411"
- board text added: "FLASH"
- board text added: "HSEC"
- board text added: "IMU"
- board text added: "INA219"
- board text added: "MISO1"
- board text added: "MISO2"
- board text added: "MISO3"
- board text added: "MISO4"
- board text added: "MISO5"
- board text added: "MISO6"
- board text added: "MOSI1"
- board text added: "MOSI2"
- board text added: "MOSI3"
- board text added: "MOSI4"
- board text added: "MOSI5"
- board text added: "MOSI6"
- board text added: "NSS1"
- board text added: "NSS2"
- board text added: "NSS3"
- board text added: "NSS4"
- board text added: "NSS5"
- board text added: "NSS6"
- board text added: "RESET"
- board text added: "RTC"
- board text added: "RX"
- board text added: "RX1"
- board text added: "RX2"
- board text added: "RX3"
- board text added: "RX4"
- board text added: "RX5"
- board text added: "RX6"
- board text added: "SCK1"
- board text added: "SCK2"
- board text added: "SCK3"
- board text added: "SCK4"
- board text added: "SCK5"
- board text added: "SCK6"
- board text added: "SCL1"
- board text added: "SCL2"
- board text added: "SDA1"
- board text added: "SDA2"
- board text added: "SWD"
- board text added: "TX"
- board text added: "TX1"
- board text added: "TX2"
- board text added: "TX3"
- board text added: "TX4"
- board text added: "TX5"
- board text added: "TX6"
- board text added: "VBAT"
- board text added: "VBUS"
- board text added: "VIN"
- board text added: "beep boop!"
- board text added: "let's not fuck up the board!"
- board text removed: "change switch? -> run drc -> finish silkscreen"
- board text removed: "ensure tp does not interfere with highspeed traces"
