File: 01_main-board/power.kicad_sch (KiCad schematic)
At the start: 36 parts, among them J4 XT30PW-M, Q1 AO3401A, U25 TPS562200, U26 TPS562200, U7 INA219AxD

Commit message: power routing
Parts:
- removed U7: INA219AxD, Package_SO:SOIC-8_3.9x4.9mm_P1.27mm, symbol Sensor_Energy:INA219AxD
- added U9: INA219AxDCN, Package_TO_SOT_SMD:SOT-23-8, symbol Sensor_Energy:INA219AxDCN
- L3: footprint Inductor_SMD:L_Changjiang_FNR4030S -> Inductor_SMD:L_Changjiang_FXL0420
Connections:
- net +3V3: now also U9.4 (VS)
- net GND: now also U9.3 (GND)
- net I2C1_SCL: now also U9.5 (SCL)
- net I2C1_SDA: now also U9.6 (SDA)
- net VBAT: now also U9.2 (IN-)
- net at R5.2: now also U9.7 (A0)
- net at J4.2 (P), R28.2: now also U9.1 (IN+)
- net at R4.2: now also U9.8 (A1)
Changed lines of the file:
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@@
+	)
+	(symbol
+		(lib_id "Sensor_Energy:INA219AxDCN")
+		(at 80.01 57.15 0)
+		(unit 1)
+		(exclude_from_sim no)
+		(in_bom yes)
+		(on_board yes)
+		(dnp no)
+		(fields_autoplaced yes)
+		(property "Reference" "U9"
+			(at 82.1533 44.45 0)
+			(effects
+				(font
+					(size 1.27 1.27)
+				)
+				(justify left)
+			)
+		)
+		(property "Value" "INA219AxDCN"
+			(at 82.1533 46.99 0)
+			(effects
+				(font
+					(size 1.27 1.27)
+				)
+				(justify left)
+			)
+		)
+		(property "Footprint" "Package_TO_SOT_SMD:SOT-23-8"
+			(at 96.52 66.04 0)
+			(effects
+				(font
+					(size 1.27 1.27)
+				)
+				(hide yes)
+			)
+		)
+		(property "Datasheet" "http://www.ti.com/lit/ds/symlink/ina219.pdf"
+			(at 88.9 59.69 0)
+			(effects
+				(font
+					(size 1.27 1.27)
+				)
+				(hide yes)
+			)
+		)
+		(property "Description" "Zero-Drift, Bidirectional Current/Power Monitor (0-26V) With I2C Interface, SOT-23-8"
+			(at 80.01 57.15 0)
+			(effects
+				(font
+					(size 1.27 1.27)
+				)
+				(hide yes)
+			)
+		)
+		(pin "3"
+		)
+		(pin "4"
+		)
+		(pin "2"
+		)
+		(pin "1"
+		)
+		(pin "6"
+		)
+		(pin "5"
+		)
+		(pin "7"
+		)
+		(pin "8"
+		)
+		(instances
+			(project ""
+				(path "/f5781173-3155-474e-950c-81192e73c9b5/e8601e63-86ce-4e79-ade3-27db572d4722"
+					(reference "U9")
+					(unit 1)
+				)
+			)
+		)
 	)
 	(symbol
@@
 			)
 		)
-		(property "Footprint" "Inductor_SMD:L_Changjiang_FNR4030S"
+		(property "Footprint" "Inductor_SMD:L_Changjiang_FXL0420"
 			(at 101.6 135.89 0)
 			(effects
@@
 					(unit 1)
 				)
-			)
-		)
-	)
-	(symbol
-		(lib_id "Sensor_Energy:INA219AxD")
-		(at 80.01 57.15 0)
-		(unit 1)
-		(exclude_from_sim no)
-		(in_bom yes)
-		(on_board yes)
-		(dnp no)
-		(fields_autoplaced yes)
-		(property "Reference" "U7"
-			(at 82.2041 44.45 0)
-			(effects
-				(font
-					(size 1.27 1.27)
-				)
-				(justify left)
-			)
-		)
-		(property "Value" "INA219AxD"
-			(at 82.2041 46.99 0)
-			(effects
-				(font
-					(size 1.27 1.27)
-				)
-				(justify left)
-			)
-		)
-		(property "Footprint" "Package_SO:SOIC-8_3.9x4.9mm_P1.27mm"
-			(at 100.33 66.04 0)
-			(effects
-				(font
-					(size 1.27 1.27)
-				)
-				(hide yes)
-			)
-		)
-		(property "Datasheet" "http://www.ti.com/lit/ds/symlink/ina219.pdf"
-			(at 88.9 59.69 0)
-			(effects
-				(font
-					(size 1.27 1.27)
-				)
-				(hide yes)
-			)
-		)
-		(property "Description" "Zero-Drift, Bidirectional Current/Power Monitor (0-26V) With I2C Interface, SOIC-8"
-			(at 80.01 57.15 0)
-			(effects
-				(font
-					(size 1.27 1.27)
-				)
-				(hide yes)
-			)
-		)
-		(pin "8"
-		)
-		(pin "1"
-		)
-		(pin "6"
-		)
-		(pin "2"
-		)
-		(pin "3"
-		)
-		(pin "4"
-		)
-		(pin "5"
-		)
-		(pin "7"
-		)
-		(instances
-			(project ""
-				(path "/f5781173-3155-474e-950c-81192e73c9b5/e8601e63-86ce-4e79-ade3-27db572d4722"
-					(reference "U7")
-					(unit 1)
-				)
