File: 01_main-board/Dumpling_Main.kicad_sch (KiCad schematic)
At the start: 55 parts, among them J1 Conn_ARM_SWD_TagConnect_TC203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, J2 Micro_SD_Card, J3 USB_C_Receptacle_USB2.0_16P, Q2 S8050, SW1 SW_SPDT, SW2 SW_DPST, U1 STM32F405RGTx, U2 USBLC6-2SC6, U8 W25Q128JVE, Y2 32.768kHz

Commit message: added coprocessors
Parts:
- removed U8: W25Q128JVE, Package_SON:WSON-8-1EP_8x6mm_P1.27mm_EP3.4x4.3mm, symbol Memory_Flash:W25Q128JVE
- added H1, H2, H3, H4: MountingHole, MountingHole:MountingHole_3.2mm_M3_Pad_Via, symbol Mechanical:MountingHole
- added U24: W25Q128JVS, Package_SO:SOIC-8_5.3x5.3mm_P1.27mm, symbol Memory_Flash:W25Q128JVS
- BZ1: footprint (none) -> CSS-0575B-SMT:CUI_CSS-0575B-SMT
- C11, C12, C3, C4: footprint Capacitor_SMD:C_0603_1608Metric -> Capacitor_SMD:C_0402_1005Metric
- C6: footprint Capacitor_SMD:C_0201_0603Metric -> Capacitor_SMD:C_0402_1005Metric
- R1: footprint (none) -> Capacitor_SMD:C_0402_1005Metric
- SW1: value SW_SPDT -> SW_DPST; footprint (none) -> CJS-1200TA:SW_CJS-1200TA
- SW2: footprint (none) -> Button_Switch_SMD:SW_SPST_B3U-1000P
- TP1, TP10, TP11, TP2, TP3, TP4, TP5, TP6, TP7, TP8, TP9: footprint (none) -> TestPoint:TestPoint_Pad_D1.0mm
- Y2: footprint (none) -> Crystal:Crystal_SMD_3215-2Pin_3.2x1.5mm
Connections:
- net +3V3: now also U24.8 (VCC)
- net FLASH_HOLD: now also R34.2, U24.7 (~{HOLD}/~{RESET}/IO_{3}); no longer R33.2, U1.15 (PA1)
- net FLASH_WP: now also R33.2, U24.3 (~{WP}/IO_{2}); no longer R34.2, U1.14 (PA0)
- net GND: now also D7.2 (VSS), U24.4 (GND)
- net SPI1_MISO: now also U24.2 (DO/IO_{1})
- net SPI1_MOSI: now also U24.5 (DI/IO_{0})
- net SPI1_NSS: now also U24.1 (~{CS})
- net SPI1_SCK: now also U24.6 (CLK)
Other:
- added sheet Coprocessor_2 (coprocessor_2.kicad_sch)
- added sheet Coprocessor_3 (coprocessor_3.kicad_sch)
- added sheet Coprocessor_4 (corprocessor_4.kicad_sch)
- added sheet Coprocessor_5 (coprocessor_5.kicad_sch)
- added sheet Coprocessor_6 (coprocessor_6.kicad_sch)
- note added: "Mounting Holes"
- moved on the sheet: TP1, TP10, TP11, TP2, TP3, TP4, TP5, TP6, TP7, TP8, TP9

Commit message: power routing
Parts:
- added J5: SM04B-SRSS-TB, Connector_JST:JST_SH_SM04B-SRSS-TB_1x04-1MP_P1.00mm_Horizontal, symbol SM04B-SRSS-TB:SM04B-SRSS-TB
- C2: footprint Capacitor_SMD:C_0201_0603Metric -> Capacitor_SMD:C_0805_2012Metric
- Q2: footprint Package_TO_SOT_THT:TO-92_Inline -> Package_TO_SOT_SMD:SOT-23
Connections:
- net GND: now also J3.S1 (SHIELD), J5.1
- net SPI2_NSS1: now also U1.11 (PC3); no longer U1.33 (PB12)
- net SPI2_NSS2: now also U1.33 (PB12); no longer U1.10 (PC2)
- net SPI2_NSS3: now also U1.10 (PC2); no longer U1.11 (PC3)
- net SPI2_NSS4: now also U1.37 (PC6); no longer U1.24 (PC4)
- net SPI2_NSS5: now also U1.24 (PC4); no longer U1.25 (PC5)
- net SPI2_NSS6: now also U1.25 (PC5); no longer U1.37 (PC6)
- net USART_RX: now also J5.3
- net USART_TX: now also J5.4
- new net +5V: J5.2
- no-connect marks 5 -> 4
Other:
- note added: "Radio"
- moved on the sheet: BZ1, C1, C11, C12, C3, C4, D7, H1, H2, H3, H4, HSE1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

Commit message: wired
Parts:
- added C105: 10n, Capacitor_SMD:C_0402_1005Metric, symbol Device:C
- added C106, C107: 0.22u, Capacitor_SMD:C_0402_1005Metric, symbol Device:C
- added R80, R81: 4.7k, Resistor_SMD:R_0402_1005Metric, symbol Device:R
- added R82, R83: 5.1k, Resistor_SMD:R_0402_1005Metric, symbol Device:R
- added R84: 10k, Resistor_SMD:R_0402_1005Metric, symbol Device:R
- added S1: JS102011JCQN, JS102011JCQN:SW_JS102011JCQN, symbol JS102011JCQN:JS102011JCQN
- added U7: MPU-6050, Sensor_Motion:InvenSense_QFN-24_4x4mm_P0.5mm, symbol Sensor_Motion:MPU-6050
Connections:
- net +3V3: now also C105.2, R80.1, R81.1, R84.2, U7.13 (VDD), U7.8 (VLOGIC)
- net GND: now also C105.1, C106.2, C107.2, R82.1, R83.1, U7.1 (CLKIN), U7.11 (FSYNC), U7.18 (GND), U7.9 (AD0)
- net SDIO_D7: now reaches U1.38 (PC7)
- net SDIO_D7: now also J2.8 (DAT1)
- net I2C3_SCL: now reaches U1.41 (PA8)
- net I2C3_SCL: now also R81.2, U7.23 (SCL)
- net IMU_INT: now reaches U1.42 (PA9)
- net IMU_INT: now also R84.1, U7.12 (INT)
- net SDIO_D1 renamed I2C3_SDA
- net I2C3_SDA: now also R80.2, U7.24 (SDA); no longer J2.8 (DAT1)
- new net: R83.2, U7.7 (AUX_CL)
- new net: C107.1, U7.20 (CPOUT)
- new net: C106.1, U7.10 (REGOUT)
- new net: R82.2, U7.6 (AUX_DA)
Other:
- note added: "I2C Address: 0x68"
- note added: "IMU"
- note added: "VLOGIC = 1.71V to VDD"
- note removed: "Radio"
- moved on the sheet: BZ1, C1, D1, D7, H1, H2, H3, H4, J5, Q2, R2, R22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

Commit message: wiring fin, pre-drc
Parts:
- removed S1: JS102011JCQN, JS102011JCQN:SW_JS102011JCQN, symbol JS102011JCQN:JS102011JCQN
Changed lines of the file:
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@@
-	)
-	(symbol
-		(lib_id "JS102011JCQN:JS102011JCQN")
-		(at 182.88 151.13 0)
-		(unit 1)
-		(exclude_from_sim no)
-		(in_bom yes)
-		(on_board yes)
-		(dnp no)
-		(fields_autoplaced yes)
-		(property "Reference" "S1"
-			(at 181.61 143.51 0)
-			(effects
-				(font
-					(size 1.27 1.27)
-				)
-			)
-		)
-		(property "Value" "JS102011JCQN"
-			(at 181.61 146.05 0)
-			(effects
-				(font
-					(size 1.27 1.27)
-				)
-			)
-		)
-		(property "Footprint" "JS102011JCQN:SW_JS102011JCQN"
-			(at 182.88 151.13 0)
-			(effects
-				(font
-					(size 1.27 1.27)
-				)
-				(justify bottom)
-				(hide yes)
-			)
-		)
-		(property "Datasheet" ""
-			(at 182.88 151.13 0)
-			(effects
-				(font
-					(size 1.27 1.27)
-				)
-				(hide yes)
-			)
-		)
-		(property "Description" ""
-			(at 182.88 151.13 0)
-			(effects
-				(font
-					(size 1.27 1.27)
-				)
-				(hide yes)
-			)
-		)
-		(property "MF" "C&K"
-			(at 182.88 151.13 0)
-			(effects
-				(font
-					(size 1.27 1.27)
-				)
-				(justify bottom)
-				(hide yes)
-			)
-		)
-		(property "Description_1" "Slide Switch SPDT Surface Mount"
-			(at 182.88 151.13 0)
-			(effects
-				(font
-					(size 1.27 1.27)
-				)
-				(justify bottom)
-				(hide yes)
-			)
-		)
-		(property "Package" "None"
-			(at 182.88 151.13 0)
-			(effects
-				(font
-					(size 1.27 1.27)
-				)
-				(justify bottom)
-				(hide yes)
-			)
-		)
-		(property "Price" "None"
-			(at 182.88 151.13 0)
-			(effects
-				(font
-					(size 1.27 1.27)
-				)
-				(justify bottom)
-				(hide yes)
-			)
-		)
-		(property "Check_prices" "https://www.snapeda.com/parts/JS102011JCQN/C%2526K/view-part/?ref=eda"
-			(at 182.88 151.13 0)
-			(effects
-				(font
-					(size 1.27 1.27)
-				)
-				(justify bottom)
-				(hide yes)
-			)
-		)
-		(property "STANDARD" "MANUFACTURER RECOMMENDATIONS"
-			(at 182.88 151.13 0)
-			(effects
-				(font
-					(size 1.27 1.27)
-				)
-				(justify bottom)
-				(hide yes)
-			)
-		)
-		(property "PARTREV" "29 JUN 2016"
-			(at 182.88 151.13 0)
-			(effects
-				(font
-					(size 1.27 1.27)
-				)
-				(justify bottom)
-				(hide yes)
-			)
-		)
-		(property "SnapEDA_Link" "https://www.snapeda.com/parts/JS102011JCQN/C%2526K/view-part/?ref=snap"
-			(at 182.88 151.13 0)
-			(effects
-				(font
-					(size 1.27 1.27)
-				)
-				(justify bottom)
-				(hide yes)
-			)
-		)
-		(property "MP" "JS102011JCQN"
-			(at 182.88 151.13 0)
-			(effects
-				(font
-					(size 1.27 1.27)
-				)
-				(justify bottom)
-				(hide yes)
-			)
-		)
-		(property "Availability" "In Stock"
-			(at 182.88 151.13 0)
-			(effects
-				(font
-					(size 1.27 1.27)
-				)
-				(justify bottom)
-				(hide yes)
-			)
-		)
-		(property "MANUFACTURER" "CK COMPONENTS"
-			(at 182.88 151.13 0)
-			(effects
-				(font
-					(size 1.27 1.27)
-				)
-				(justify bottom)
-				(hide yes)
-			)
-		)
-		(pin "1"
-		)
-		(pin "3"
-		)
-		(pin "2"
-		)
-		(instances
-			(project ""
-				(path "/f5781173-3155-474e-950c-81192e73c9b5"
-					(reference "S1")
-					(unit 1)
-				)
-			)
-		)
 	)
 	(symbol

Commit message: ebay backboard
Parts:
- BZ1: footprint CSS-0575B-SMT:CUI_CSS-0575B-SMT -> FST-5030:BUZ-SMD_FST-5030
- SW1: value SW_DPST -> SW_SPDT; footprint CJS-1200TA:SW_CJS-1200TA -> JS102011JCQN:SW_JS102011JCQN
- SW2: value SW_DPST -> SW_SPST
Connections:
- no-connect marks 4 -> 6
Changed lines of the file:
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@@
 	)
 	(no_connect
+		(at 31.75 100.33)
+	)
+	(no_connect
 		(at 165.1 38.1)
 	)
@@
 		(at 256.54 54.61)
 	)
+	(no_connect
+		(at 31.75 93.98)
+	)
 	(wire
 		(pts
@@
 			)
 		)
-		(property "Value" "SW_DPST"
+		(property "Value" "SW_SPST"
 			(at 176.53 123.444 0)
 			(effects
@@
 			)
 		)
-		(property "Value" "SW_DPST"
+		(property "Value" "SW_SPDT"
 			(at 128.27 107.442 0)
 			(effects
@@
 			)
 		)
-		(property "Footprint" "CJS-1200TA:SW_CJS-1200TA"
+		(property "Footprint" "JS102011JCQN:SW_JS102011JCQN"
 			(at 128.27 113.03 0)
 			(effects
@@
 			)
 		)
-		(property "Footprint" "CSS-0575B-SMT:CUI_CSS-0575B-SMT"
+		(property "Footprint" "FST-5030:BUZ-SMD_FST-5030"
 			(at 95.885 135.89 90)
 			(effects
