File: 01_main-board/coprocessor_1.kicad_sch (KiCad schematic)
At the start: 43 parts, among them J7 MICROMOD-2222-C, J8 USB_C_Receptacle_USB2.0_16P, J9 Conn_ARM_SWD_TagConnect_TC203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, SW3 SW_DPST, SW4 SW_SPDT, U3 W25Q128JVS, U4 STM32F411CEUx, U6 USBLC6-2SC6, Y1 32.768kHz

Commit message: power routing
Connections:
- net GND: now also J8.S1 (SHIELD)
- net co1_RGB_LED: no longer J7.40 (G0/BUS0)
- net co1_SPI3_MISO: now also J7.62 (SPI_SDO1/SDIO_CMD); no longer J7.59 (SPI_SDO)
- net co1_SPI3_MOSI: now also J7.60 (SPI_SDI1/SDIO_DATA0); no longer J7.61 (SPI_SDI)
- net co1_SPI3_NSS: now also J7.66 (SPI_~{CS1}/SDIO_DATA3)
- net co1_SPI3_SCK: now also J7.64 (SPI_SCK1/SDIO_CLK); no longer J7.57 (SPI_SCK)
- net co1_SPI3_NSS1: no longer names the net of J7.55 (SPI_~{CS})
- no-connect marks 4 -> 3
Changed lines of the file:
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@@
 	)
 	(no_connect
-		(at 125.73 160.02)
-	)
-	(no_connect
 		(at 176.53 105.41)
 	)
@@
 	(wire
 		(pts
-			(xy 219.71 160.02) (xy 219.71 156.21)
-		)
-		(stroke
-			(width 0)
-			(type default)
-		)
-	)
-	(wire
-		(pts
 			(xy 52.07 110.49) (xy 54.61 110.49)
 		)
@@
 	(wire
 		(pts
-			(xy 218.44 160.02) (xy 218.44 161.29)
+			(xy 218.44 156.21) (xy 218.44 161.29)
 		)
 		(stroke
@@
 	(wire
 		(pts
+			(xy 218.44 156.21) (xy 219.71 156.21)
+		)
+		(stroke
+			(width 0)
+			(type default)
+		)
+	)
+	(wire
+		(pts
 			(xy 160.02 69.85) (xy 160.02 71.12)
 		)
@@
 	(wire
 		(pts
+			(xy 125.73 158.75) (xy 125.73 160.02)
+		)
+		(stroke
+			(width 0)
+			(type default)
+		)
+	)
+	(wire
+		(pts
 			(xy 115.57 63.5) (xy 120.65 63.5)
 		)
@@
 		)
 	)
-	(wire
-		(pts
-			(xy 219.71 160.02) (xy 218.44 160.02)
-		)
-		(stroke
-			(width 0)
-			(type default)
-		)
-	)
 	(global_label "co1_SPI1_MOSI"
 		(shape input)
@@
 		)
 	)
-	(global_label "co1_SPI3_MISO"
-		(shape input)
-		(at 265.43 100.33 0)
-		(fields_autoplaced yes)
-		(effects
-			(font
-				(size 1.27 1.27)
-			)
-			(justify left)
-		)
-		(property "Intersheetrefs" "${INTERSHEET_REFS}"
-			(at 282.6875 100.33 0)
-			(effects
-				(font
-					(size 1.27 1.27)
-				)
-				(justify left)
-				(hide yes)
-			)
-		)
-	)
 	(global_label "VBUS"
 		(shape input)
@@
 		)
 	)
+	(global_label "co1_SPI3_SCK"
+		(shape input)
+		(at 265.43 99.06 0)
+		(fields_autoplaced yes)
+		(effects
+			(font
+				(size 1.27 1.27)
+				(thickness 0.1588)
+			)
+			(justify left)
+		)
+		(property "Intersheetrefs" "${INTERSHEET_REFS}"
+			(at 281.8408 99.06 0)
+			(effects
+				(font
+					(size 1.27 1.27)
+				)
+				(justify left)
+				(hide yes)
+			)
+		)
+	)
 	(global_label "co1_gpio2"
 		(shape input)
@@
 		)
 	)
+	(global_label "co1_SPI3_NSS"
+		(shape input)
+		(at 265.43 96.52 0)
+		(fields_autoplaced yes)
+		(effects
+			(font
+				(size 1.27 1.27)
+				(thickness 0.1588)
+			)
+			(justify left)
+		)
+		(property "Intersheetrefs" "${INTERSHEET_REFS}"
+			(at 281.8408 96.52 0)
+			(effects
+				(font
+					(size 1.27 1.27)
+				)
+				(justify left)
+				(hide yes)
+			)
+		)
+	)
 	(global_label "co1_USART_RX"
 		(shape input)
@@
 		)
 	)
-	(global_label "co1_RGB_LED"
+	(global_label "co1_SPI3_SCK"
 		(shape input)
-		(at 265.43 128.27 0)
+		(at 69.85 64.77 0)
 		(fields_autoplaced yes)
 		(effects
@@
 		)
 		(property "Intersheetrefs" "${INTERSHEET_REFS}"
-			(at 281.0546 128.27 0)
+			(at 86.2608 64.77 0)
 			(effects
 				(font
@@
 		)
 	)
-	(global_label "co1_SPI3_SCK"
+	(global_label "co1_SPI1_SCK"
 		(shape input)
-		(at 69.85 64.77 0)
+		(at 185.42 66.04 180)
 		(fields_autoplaced yes)
 		(effects
@@
 				(size 1.27 1.27)
 			)
-			(justify left)
+			(justify right)
 		)
 		(property "Intersheetrefs" "${INTERSHEET_REFS}"
-			(at 86.2608 64.77 0)
+			(at 169.0092 66.04 0)
 			(effects
 				(font
 					(size 1.27 1.27)
 				)
-				(justify left)
+				(justify right)
 				(hide yes)
 			)
 		)
 	)
-	(global_label "co1_SPI1_SCK"
+	(global_label "co1_SPI3_MOSI"
 		(shape input)
-		(at 185.42 66.04 180)
+		(at 265.43 104.14 0)
 		(fields_autoplaced yes)
 		(effects
@@
 				(size 1.27 1.27)
 			)
-			(justify right)
+			(justify left)
 		)
 		(property "Intersheetrefs" "${INTERSHEET_REFS}"
-			(at 169.0092 66.04 0)
+			(at 282.6875 104.14 0)
 			(effects
 				(font
 					(size 1.27 1.27)
 				)
-				(justify right)
+				(justify left)
 				(hide yes)
 			)
@@
 		)
 	)
-	(global_label "co1_SPI3_SCK"
-		(shape input)
-		(at 265.43 97.79 0)
-		(fields_autoplaced yes)
-		(effects
-			(font
-				(size 1.27 1.27)
-				(thickness 0.1588)
-			)
-			(justify left)
-		)
-		(property "Intersheetrefs" "${INTERSHEET_REFS}"
-			(at 281.8408 97.79 0)
-			(effects
-				(font
-					(size 1.27 1.27)
-				)
-				(justify left)
-				(hide yes)
-			)
-		)
-	)
 	(global_label "co1_FLASH_WP"
 		(shape input)
@@
 		)
 	)
+	(global_label "co1_SPI3_MISO"
+		(shape input)
+		(at 265.43 101.6 0)
+		(fields_autoplaced yes)
+		(effects
+			(font
+				(size 1.27 1.27)
+			)
+			(justify left)
+		)
+		(property "Intersheetrefs" "${INTERSHEET_REFS}"
+			(at 282.6875 101.6 0)
+			(effects
+				(font
+					(size 1.27 1.27)
+				)
+				(justify left)
+				(hide yes)
+			)
+		)
+	)
 	(global_label "co1_NRST"
 		(shape input)
@@
 		)
 	)
-	(global_label "co1_SPI3_MOSI"
-		(shape input)
-		(at 265.43 102.87 0)
-		(fields_autoplaced yes)
-		(effects
-			(font
-				(size 1.27 1.27)
-			)
-			(justify left)
-		)
-		(property "Intersheetrefs" "${INTERSHEET_REFS}"
-			(at 282.6875 102.87 0)
-			(effects
-				(font
-					(size 1.27 1.27)
-				)
-				(justify left)
-				(hide yes)
-			)
-		)
-	)
 	(global_label "co1_RTC_IN"
 		(shape input)
@@
 		)
 	)
-	(global_label "co1_SPI3_NSS1"
-		(shape input)
-		(at 265.43 105.41 0)
-		(fields_autoplaced yes)
-		(effects
-			(font
-				(size 1.27 1.27)
-				(thickness 0.1588)
-			)
-			(justify left)
-		)
-		(property "Intersheetrefs" "${INTERSHEET_REFS}"
-			(at 283.0503 105.41 0)
-			(effects
-				(font
-					(size 1.27 1.27)
-				)
-				(justify left)
-				(hide yes)
-			)
-		)
-	)
 	(global_label "co1_RGB_LED"
 		(shape input)
@@
 					(unit 1)
 				)
+			)
+		)
+	)
+	(symbol
+		(lib_id "power:GND")
+		(at 125.73 158.75 0)
+		(unit 1)
+		(exclude_from_sim no)
+		(in_bom yes)
+		(on_board yes)
+		(dnp no)
+		(property "Reference" "#PWR0223"
+			(at 125.73 165.1 0)
+			(effects
+				(font
+					(size 1.27 1.27)
+				)
+				(hide yes)
+			)
+		)
+		(property "Value" "GND"
+			(at 131.826 160.782 0)
+			(effects
+				(font
+					(size 1.27 1.27)
+				)
+				(justify right)
+			)
+		)
+		(property "Footprint" ""
+			(at 125.73 158.75 0)
+			(effects
+				(font
+					(size 1.27 1.27)
+				)
+				(hide yes)
+			)
+		)
+		(property "Datasheet" ""
+			(at 125.73 158.75 0)
+			(effects
+				(font
+					(size 1.27 1.27)
+				)
+				(hide yes)
+			)
+		)
+		(property "Description" "Power symbol creates a global label with name \"GND\" , ground"
+			(at 125.73 158.75 0)
+			(effects
+				(font
+					(size 1.27 1.27)
+				)
+				(hide yes)
+			)
+		)
+		(pin "1"
+		)
+		(instances
+			(project "Dumpling_Main"
+				(path "/f5781173-3155-474e-950c-81192e73c9b5/e6b2dda1-d2a7-47da-9e5f-a024a9da6110"
+					(reference "#PWR0223")
+					(unit 1)
+				)

Commit message: ebay backboard
Parts:
- removed MP1: ~, WA-SMSI_9774XXX151:WA-SMSI_9774025151, symbol WA-SMSI_9774XXX151:WA-SMSI_9774XXX151
- added U21: SMTSOM2_525STR, SMTSOM2.525STR:SMD_BD5.6-D4.1, symbol SMTSOM2_525STR:SMTSOM2_525STR
- SW3: value SW_DPST -> SW_SPST
- SW4: footprint CJS-1200TA:SW_CJS-1200TA -> JS102011JCQN:SW_JS102011JCQN
Connections:
- net GND: now also U21.1, U21.2, U21.3, U21.4
- net at J8.A8 (SBU1): no longer J8.B8 (SBU2)
- no-connect marks 3 -> 48
Other:
- note added: "Standoff (Patch round nut)"
- note removed: "WA-SMSI_9774XXX151"
