File: 01_main-board/coprocessor_2.kicad_sch (KiCad schematic)
At the start: 43 parts, among them J10 MICROMOD-2222-C, J23 USB_C_Receptacle_USB2.0_16P, J6 Conn_ARM_SWD_TagConnect_TC203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, SW5 SW_DPST, SW6 SW_SPDT, U11 USBLC6-2SC6, U5 STM32F411CEUx, U8 W25Q128JVS, Y3 32.768kHz

Commit message: power routing
Connections:
- net GND: now also J23.S1 (SHIELD)
- net co2_RGB_LED: no longer J10.40 (G0/BUS0)
- net co2_SPI3_MISO: now also J10.62 (SPI_SDO1/SDIO_CMD); no longer J10.59 (SPI_SDO)
- net co2_SPI3_MOSI: now also J10.60 (SPI_SDI1/SDIO_DATA0); no longer J10.61 (SPI_SDI)
- net co2_SPI3_NSS: now also J10.66 (SPI_~{CS1}/SDIO_DATA3)
- net co2_SPI3_SCK: now also J10.64 (SPI_SCK1/SDIO_CLK); no longer J10.57 (SPI_SCK)
- net co2_SPI3_NSS1: no longer names the net of J10.55 (SPI_~{CS})
- no-connect marks 4 -> 3

Commit message: ebay backboard
Parts:
- removed MP2: ~, WA-SMSI_9774XXX151:WA-SMSI_9774025151, symbol WA-SMSI_9774XXX151:WA-SMSI_9774XXX151
- added U27: SMTSOM2_525STR, SMTSOM2.525STR:SMD_BD5.6-D4.1, symbol SMTSOM2_525STR:SMTSOM2_525STR
- SW5: value SW_DPST -> SW_SPST
- SW6: footprint CJS-1200TA:SW_CJS-1200TA -> JS102011JCQN:SW_JS102011JCQN
Connections:
- net GND: now also U27.1, U27.2, U27.3, U27.4
- net at J23.A8 (SBU1): no longer J23.B8 (SBU2)
- no-connect marks 3 -> 48
Other:
- note added: "Standoff (Patch round nut)"
