File: 01_main-board/coprocessor_3.kicad_sch (KiCad schematic)
At the start: 43 parts, among them J11 USB_C_Receptacle_USB2.0_16P, J12 Conn_ARM_SWD_TagConnect_TC203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, J13 MICROMOD-2222-C, SW7 SW_DPST, SW8 SW_SPDT, U10 W25Q128JVS, U13 STM32F411CEUx, U14 USBLC6-2SC6, Y4 32.768kHz

Commit message: power routing
Connections:
- net GND: now also J11.S1 (SHIELD)
- net co3_RGB_LED: no longer J13.40 (G0/BUS0)
- net co3_SPI3_MISO: now also J13.62 (SPI_SDO1/SDIO_CMD); no longer J13.59 (SPI_SDO)
- net co3_SPI3_MOSI: now also J13.60 (SPI_SDI1/SDIO_DATA0); no longer J13.61 (SPI_SDI)
- net co3_SPI3_NSS: now also J13.66 (SPI_~{CS1}/SDIO_DATA3)
- net co3_SPI3_SCK: now also J13.64 (SPI_SCK1/SDIO_CLK); no longer J13.57 (SPI_SCK)
- net co3_SPI3_NSS1: no longer names the net of J13.55 (SPI_~{CS})
- no-connect marks 4 -> 3

Commit message: ebay backboard
Parts:
- removed MP3: ~, WA-SMSI_9774XXX151:WA-SMSI_9774025151, symbol WA-SMSI_9774XXX151:WA-SMSI_9774XXX151
- added U28: SMTSOM2_525STR, SMTSOM2.525STR:SMD_BD5.6-D4.1, symbol SMTSOM2_525STR:SMTSOM2_525STR
- SW7: value SW_DPST -> SW_SPST
- SW8: footprint CJS-1200TA:SW_CJS-1200TA -> JS102011JCQN:SW_JS102011JCQN
Connections:
- net GND: now also U28.1, U28.2, U28.3, U28.4
- net at J11.A8 (SBU1): no longer J11.B8 (SBU2)
- no-connect marks 3 -> 47
Other:
- note added: "Standoff (Patch round nut)"
