File: 01_main-board/coprocessor_5.kicad_sch (KiCad schematic)
At the start: 43 parts, among them J17 USB_C_Receptacle_USB2.0_16P, J18 Conn_ARM_SWD_TagConnect_TC203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, J19 MICROMOD-2222-C, SW11 SW_DPST, SW12 SW_SPDT, U15 W25Q128JVS, U19 STM32F411CEUx, U20 USBLC6-2SC6, Y6 32.768kHz

Commit message: power routing
Connections:
- net GND: now also J17.S1 (SHIELD)
- net co5_RGB_LED: no longer J19.40 (G0/BUS0)
- net co5_SPI3_MISO: now also J19.62 (SPI_SDO1/SDIO_CMD); no longer J19.59 (SPI_SDO)
- net co5_SPI3_MOSI: now also J19.60 (SPI_SDI1/SDIO_DATA0); no longer J19.61 (SPI_SDI)
- net co5_SPI3_NSS: now also J19.66 (SPI_~{CS1}/SDIO_DATA3)
- net co5_SPI3_SCK: now also J19.64 (SPI_SCK1/SDIO_CLK); no longer J19.57 (SPI_SCK)
- net co5_SPI3_NSS1: no longer names the net of J19.55 (SPI_~{CS})
- no-connect marks 4 -> 3

Commit message: ebay backboard
Parts:
- removed MP5: ~, WA-SMSI_9774XXX151:WA-SMSI_9774025151, symbol WA-SMSI_9774XXX151:WA-SMSI_9774XXX151
- added U30: SMTSOM2_525STR, SMTSOM2.525STR:SMD_BD5.6-D4.1, symbol SMTSOM2_525STR:SMTSOM2_525STR
- SW11: value SW_DPST -> SW_SPST
- SW12: footprint CJS-1200TA:SW_CJS-1200TA -> JS102011JCQN:SW_JS102011JCQN
Connections:
- net GND: now also U30.1, U30.2, U30.3, U30.4
- net at J17.A8 (SBU1): no longer J17.B8 (SBU2)
- no-connect marks 3 -> 48
Other:
- note added: "Standoff (Patch round nut)"
