File: 01_main-board/coprocessor_6.kicad_sch (KiCad schematic)
At the start: 43 parts, among them J20 USB_C_Receptacle_USB2.0_16P, J21 Conn_ARM_SWD_TagConnect_TC203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, J22 MICROMOD-2222-C, SW13 SW_DPST, SW14 SW_SPDT, U18 W25Q128JVS, U22 STM32F411CEUx, U23 USBLC6-2SC6, Y7 32.768kHz

Commit message: power routing
Connections:
- net GND: now also J20.S1 (SHIELD)
- net co6_RGB_LED: no longer J22.40 (G0/BUS0)
- net co6_SPI3_MISO: now also J22.62 (SPI_SDO1/SDIO_CMD); no longer J22.59 (SPI_SDO)
- net co6_SPI3_MOSI: now also J22.60 (SPI_SDI1/SDIO_DATA0); no longer J22.61 (SPI_SDI)
- net co6_SPI3_NSS: now also J22.66 (SPI_~{CS1}/SDIO_DATA3)
- net co6_SPI3_SCK: now also J22.64 (SPI_SCK1/SDIO_CLK); no longer J22.57 (SPI_SCK)
- net co6_SPI3_NSS1: no longer names the net of J22.55 (SPI_~{CS})
- no-connect marks 4 -> 3

Commit message: ebay backboard
Parts:
- removed MP6: ~, WA-SMSI_9774XXX151:WA-SMSI_9774025151, symbol WA-SMSI_9774XXX151:WA-SMSI_9774XXX151
- added U31: SMTSOM2_525STR, SMTSOM2.525STR:SMD_BD5.6-D4.1, symbol SMTSOM2_525STR:SMTSOM2_525STR
- SW13: value SW_DPST -> SW_SPST
- SW14: footprint CJS-1200TA:SW_CJS-1200TA -> JS102011JCQN:SW_JS102011JCQN
Connections:
- net GND: now also U31.1, U31.2, U31.3, U31.4
- net at J20.A8 (SBU1): no longer J20.B8 (SBU2)
- no-connect marks 3 -> 48
Other:
- note added: "Standoff (Patch round nut)"
