File: 01_main-board/corprocessor_4.kicad_sch (KiCad schematic)
At the start: 43 parts, among them J14 USB_C_Receptacle_USB2.0_16P, J15 Conn_ARM_SWD_TagConnect_TC203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, J16 MICROMOD-2222-C, SW10 SW_SPDT, SW9 SW_DPST, U12 W25Q128JVS, U16 STM32F411CEUx, U17 USBLC6-2SC6, Y5 32.768kHz

Commit message: power routing
Connections:
- net GND: now also J14.S1 (SHIELD)
- net co4_RGB_LED: no longer J16.40 (G0/BUS0)
- net co4_SPI3_MISO: now also J16.62 (SPI_SDO1/SDIO_CMD); no longer J16.59 (SPI_SDO)
- net co4_SPI3_MOSI: now also J16.60 (SPI_SDI1/SDIO_DATA0); no longer J16.61 (SPI_SDI)
- net co4_SPI3_NSS: now also J16.66 (SPI_~{CS1}/SDIO_DATA3)
- net co4_SPI3_SCK: now also J16.64 (SPI_SCK1/SDIO_CLK); no longer J16.57 (SPI_SCK)
- net co4_SPI3_NSS1: no longer names the net of J16.55 (SPI_~{CS})
- no-connect marks 4 -> 3

Commit message: ebay backboard
Parts:
- removed MP4: ~, WA-SMSI_9774XXX151:WA-SMSI_9774025151, symbol WA-SMSI_9774XXX151:WA-SMSI_9774XXX151
- added U29: SMTSOM2_525STR, SMTSOM2.525STR:SMD_BD5.6-D4.1, symbol SMTSOM2_525STR:SMTSOM2_525STR
- SW10: footprint CJS-1200TA:SW_CJS-1200TA -> JS102011JCQN:SW_JS102011JCQN
- SW9: value SW_DPST -> SW_SPST
Connections:
- net GND: now also U29.1, U29.2, U29.3, U29.4
- net at J14.A8 (SBU1): no longer J14.B8 (SBU2)
- no-connect marks 3 -> 48
Other:
- note added: "Standoff (Patch round nut)"
