File: 02_03_sensor_IMU_BMI088/02_03_sensor_IMU_BMI088.kicad_pcb (KiCad board)
At the start: 2 copper layers, 22 x 22 mm, 17 parts, among them J1 MICROMOD-2222, U1 BMI088, U2 AP2112K-3.3

Commit message: filled missing connections :/
Parts:
- U2: value AP2112K-3.3 -> TPSPX3819M5-L-3-3; footprint Package_TO_SOT_SMD:SOT-23-5 -> TPSPX3819M5-L-3-3:SOT-23-5_L3.0-W1.6-P0.95-LS2.8-BR
- moved U2 0.06 mm to (153.4, 104.6), turned to 0 degrees
- renumbered MISO to MISO1, MOSI to MOSI1, SCK to SCK1
