File: 02_04_sensor_barometer_BMP390L/02_04_sensor_barometer_BMP390L.kicad_sch (KiCad schematic)
At the start: 12 parts, among them J1 MICROMOD-2222, U1 BMP390L, U2 AP2112K-3.3

Commit message: filled missing connections :/
Parts:
- removed U2: AP2112K-3.3, Package_TO_SOT_SMD:SOT-23-5, symbol Regulator_Linear:AP2112K-3.3
- added U2: TPSPX3819M5-L-3-3, TPSPX3819M5-L-3-3:SOT-23-5_L3.0-W1.6-P0.95-LS2.8-BR, symbol TPSPX3819M5-L-3-3:TPSPX3819M5-L-3-3
Connections:
- net +3V3: now also U2.5 (VOUT)
- net GND: now also U2.2 (GND)
- net VIN: now also U2.1 (VIN), U2.3 (EN)
- no-connect marks 52 -> 53
Other:
- note added: "Address: 111011X (Connect to VSS: X=0 (0x76) Connect to VDDIO: X=1 (0x77) )"
- note removed: "Address: 111011X (Connect to VSS: X=0 Connect to VDDIO: X=1)"
- moved on the sheet: C3, C4, D1, R1
