File: 02_05_sensor_magnetometer_LIS2MDLTR/02_05_sensor_magnetometer_LIS2MDLTR.kicad_pcb (KiCad board)
At the start: 2 copper layers, 22 x 22 mm, 16 parts, among them J1 MICROMOD-2222, U2 AP2112K-3.3, U3 LIS2MDLTR

Commit message: filled missing connections :/
Parts:
- U2: value AP2112K-3.3 -> TPSPX3819M5-L-3-3; footprint Package_TO_SOT_SMD:SOT-23-5 -> TPSPX3819M5-L-3-3:SOT-23-5_L3.0-W1.6-P0.95-LS2.8-BR
- turned U2 to 0 degrees
- renumbered SCL to SCL1, SDA to SDA1
