File: 02_06_sensor_temphumid_HDC3022DEJR/02_06_sensor_temphumid_HDC3022DEJR.kicad_pcb (KiCad board)
At the start: 2 copper layers, 22 x 22 mm, 17 parts, among them J1 MICROMOD-2222, U1 HDC3022DEJR, U2 AP2112K-3.3

Commit message: filled missing connections :/
Parts:
- U2: value AP2112K-3.3 -> TPSPX3819M5-L-3-3; footprint Package_TO_SOT_SMD:SOT-23-5 -> TPSPX3819M5-L-3-3:SOT-23-5_L3.0-W1.6-P0.95-LS2.8-BR
- turned U2 to 0 degrees
- renumbered ADDR0 to JP1, ADDR1 to JP2, SCL to SCL1, SDA to SDA1
