File: 02_sensor-board/02_05_magnetometer_LIS2MDLTR_I2C/02_05_magnetometer_LIS2MDLTR_I2C.kicad_sch (KiCad schematic)
At the start: 13 parts, among them J1 MICROMOD-2222, U2 TPSPX3819M5-L-3-3, U3 LIS2MDLTR

Commit message: sensor config
Other:
- note added: "I2C Address: 0x1E"
Changed lines of the file:
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@@
+		)
+	)
+	(text "I2C Address: 0x1E"
+		(exclude_from_sim no)
+		(at 75.946 81.026 0)
+		(effects
+			(font
+				(size 0.762 0.762)
+			)
 		)
 	)
